File: PCB/juny co2 Hackpad.kicad_pcb (KiCad board)
At the start: 2 copper layers, 67.9 x 59.7 mm, 14 parts, among them J1 Conn_01x04, SW1 SW_Push, SW10 RotaryEncoder_Switch, SW4 SW_Push, SW5 SW_Push, SW6 SW_Push, U1 XIAO-RP2040-SMD

Commit message: Add files via upload
Parts:
- D2, D3, D4, D5, D8, D9: footprint LED_SMD:LED_SK6812MINI_PLCC4_3.5x3.5mm_P1.75mm -> Hackclub Footprints:MX_SK6812MINI-E_REV
