File: PCB/Juny co2 Hackpad.kicad_sch (KiCad schematic)
At the start: 14 parts, among them J1 Conn_01x04, SW1 SW_Push, SW10 RotaryEncoder_Switch, SW4 SW_Push, SW5 SW_Push, SW6 SW_Push, U1 XIAO-RP2040-SMD

Commit message: Add files via upload
Parts:
- R1: value R -> 220Ω
Changed lines of the file:
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@@
 			)
 		)
-		(property "Value" "R"
+		(property "Value" "220Ω"
 			(at 55.88 34.2899 0)
 			(effects
